Commit message: fix: 22 & 24 .h .cpp error

File: ros2_ws/src/DH116_L_URDF/DH116-L000-A1/urdf/DH116-L000-A1.urdf (robot description, URDF)
Before this commit: robot DH116-L000-A1, 17 links, 16 joints
Links:
- removed link base_link
- removed link finger11_Link
- removed link finger12_Link
- removed link finger13_Link
- removed link finger14_Link
- removed link finger21_Link
- removed link finger22_Link
- removed link finger23_Link
- removed link finger31_Link
- removed link finger32_Link
- removed link finger33_Link
- removed link finger41_Link
- removed link finger42_Link
- removed link finger43_Link
- removed link finger51_Link
- removed link finger52_Link
- removed link finger53_Link
- added link L_base_link, mass 0.11674; collision mesh filename=L_package://DH116-L000-A1/meshes/base_link.STL; visual mesh filename=L_package://DH116-L000-A1/meshes/base_link.STL
- added link L_finger11_Link, mass 0.010254; collision mesh filename=L_package://DH116-L000-A1/meshes/finger11_Link.STL; visual mesh filename=L_package://DH116-L000-A1/meshes/finger11_Link.STL
- added link L_finger12_Link, mass 0.010117; collision mesh filename=L_package://DH116-L000-A1/meshes/finger12_Link.STL; visual mesh filename=L_package://DH116-L000-A1/meshes/finger12_Link.STL
- added link L_finger13_Link, mass 0.020548; collision mesh filename=L_package://DH116-L000-A1/meshes/finger13_Link.STL; visual mesh filename=L_package://DH116-L000-A1/meshes/finger13_Link.STL
- added link L_finger14_Link, mass 0.00063385; collision mesh filename=L_package://DH116-L000-A1/meshes/finger14_Link.STL; visual mesh filename=L_package://DH116-L000-A1/meshes/finger14_Link.STL
- added link L_finger21_Link, mass 0.0067138; collision mesh filename=L_package://DH116-L000-A1/meshes/finger21_Link.STL; visual mesh filename=L_package://DH116-L000-A1/meshes/finger21_Link.STL
- added link L_finger22_Link, mass 0.014791; collision mesh filename=L_package://DH116-L000-A1/meshes/finger22_Link.STL; visual mesh filename=L_package://DH116-L000-A1/meshes/finger22_Link.STL
- added link L_finger23_Link, mass 0.00081811; collision mesh filename=L_package://DH116-L000-A1/meshes/finger23_Link.STL; visual mesh filename=L_package://DH116-L000-A1/meshes/finger23_Link.STL
- added link L_finger31_Link, mass 0.0067137; collision mesh filename=L_package://DH116-L000-A1/meshes/finger31_Link.STL; visual mesh filename=L_package://DH116-L000-A1/meshes/finger31_Link.STL
- added link L_finger32_Link, mass 0.017437; collision mesh filename=L_package://DH116-L000-A1/meshes/finger32_Link.STL; visual mesh filename=L_package://DH116-L000-A1/meshes/finger32_Link.STL
- added link L_finger33_Link, mass 0.00081807; collision mesh filename=L_package://DH116-L000-A1/meshes/finger33_Link.STL; visual mesh filename=L_package://DH116-L000-A1/meshes/finger33_Link.STL
- added link L_finger41_Link, mass 0.0067137; collision mesh filename=L_package://DH116-L000-A1/meshes/finger41_Link.STL; visual mesh filename=L_package://DH116-L000-A1/meshes/finger41_Link.STL
- added link L_finger42_Link, mass 0.014791; collision mesh filename=L_package://DH116-L000-A1/meshes/finger42_Link.STL; visual mesh filename=L_package://DH116-L000-A1/meshes/finger42_Link.STL
- added link L_finger43_Link, mass 0.00081812; collision mesh filename=L_package://DH116-L000-A1/meshes/finger43_Link.STL; visual mesh filename=L_package://DH116-L000-A1/meshes/finger43_Link.STL
- added link L_finger51_Link, mass 0.0067139; collision mesh filename=L_package://DH116-L000-A1/meshes/finger51_Link.STL; visual mesh filename=L_package://DH116-L000-A1/meshes/finger51_Link.STL
- added link L_finger52_Link, mass 0.010439; collision mesh filename=L_package://DH116-L000-A1/meshes/finger52_Link.STL; visual mesh filename=L_package://DH116-L000-A1/meshes/finger52_Link.STL
- added link L_finger53_Link, mass 0.00058044; collision mesh filename=L_package://DH116-L000-A1/meshes/finger53_Link.STL; visual mesh filename=L_package://DH116-L000-A1/meshes/finger53_Link.STL
Joints:
- removed joint finger11
- removed joint finger12
- removed joint finger13
- removed joint finger14
- removed joint finger21
- removed joint finger22
- removed joint finger23
- removed joint finger31
- removed joint finger32
- removed joint finger33
- removed joint finger41
- removed joint finger42
- removed joint finger43
- removed joint finger51
- removed joint finger52
- removed joint finger53
- added joint L_finger11: type revolute, parent L_base_link, child L_finger11_Link, origin xyz=0.018 -0.021464 0.040041 rpy=0.087266 0 0, axis 0 0 1, limit lower=-1.57 upper=1.57 effort=0 velocity=0
- added joint L_finger12: type revolute, parent L_finger11_Link, child L_finger12_Link, origin xyz=0.018876 -0.0049375 -0.0023593 rpy=0 0.95149 -0.25585, axis 0 -1 0, limit lower=0 upper=1.57 effort=0 velocity=0
- added joint L_finger13: type revolute, parent L_finger12_Link, child L_finger13_Link, origin xyz=0 0 0.045 rpy=0 0 0, axis 0 -1 0, limit lower=0 upper=1.57 effort=0 velocity=0
- added joint L_finger14: type fixed, parent L_finger13_Link, child L_finger14_Link, origin xyz=0 0 0 rpy=0 0 0, axis 0 0 0, limit lower=0 upper=1.57 effort=0 velocity=0
- added joint L_finger21: type revolute, parent L_base_link, child L_finger21_Link, origin xyz=-0.011581 -0.031971 0.10003 rpy=0.052657 0.10625 0.0055894, axis 0 1 0, limit lower=0 upper=1.57 effort=0 velocity=0
- added joint L_finger22: type revolute, parent L_finger21_Link, child L_finger22_Link, origin xyz=0 0 0.035 rpy=0 0 0, axis 0 1 0, limit lower=0 upper=1.57 effort=0 velocity=0
- added joint L_finger23: type fixed, parent L_finger22_Link, child L_finger23_Link, origin xyz=0 0 0 rpy=0 0 0, axis 0 0 0, limit lower=0 upper=1.57 effort=0 velocity=0
- added joint L_finger31: type revolute, parent L_base_link, child L_finger31_Link, origin xyz=-0.013501 -0.0105 0.10286 rpy=0 0.10214 0, axis 0 1 0, limit lower=0 upper=1.57 effort=0 velocity=0
- added joint L_finger32: type revolute, parent L_finger31_Link, child L_finger32_Link, origin xyz=0 0 0.035 rpy=0 0 0, axis 0 1 0, limit lower=0 upper=1.57 effort=0 velocity=0
- added joint L_finger33: type fixed, parent L_finger32_Link, child L_finger33_Link, origin xyz=0 0 0 rpy=0 0 0, axis 0 0 0, limit lower=0 upper=1.57 effort=0 velocity=0
- added joint L_finger41: type revolute, parent L_base_link, child L_finger41_Link, origin xyz=-0.015081 0.010971 0.10183 rpy=-0.052889 0.14148 -0.0074648, axis 0 1 0, limit lower=0 upper=1.57 effort=0 velocity=0
- added joint L_finger42: type revolute, parent L_finger41_Link, child L_finger42_Link, origin xyz=0 0 0.035 rpy=0 0 0, axis 0 1 0, limit lower=0 upper=1.57 effort=0 velocity=0
- added joint L_finger43: type fixed, parent L_finger42_Link, child L_finger43_Link, origin xyz=0 0 0 rpy=0 0 0, axis 0 0 0, limit lower=0 upper=1.57 effort=0 velocity=0
- added joint L_finger51: type revolute, parent L_base_link, child L_finger51_Link, origin xyz=-0.013081 0.032156 0.097798 rpy=-0.078754 0.073706 -0.0058113, axis 0 1 0, limit lower=0 upper=1.57 effort=0 velocity=0
- added joint L_finger52: type revolute, parent L_finger51_Link, child L_finger52_Link, origin xyz=0 0 0.035 rpy=0 0 0, axis 0 1 0, limit lower=0 upper=1.57 effort=0 velocity=0
- added joint L_finger53: type fixed, parent L_finger52_Link, child L_finger53_Link, origin xyz=0 0 0 rpy=0 0 0, axis 0 0 0, limit lower=0 upper=1.57 effort=0 velocity=0

File: ros2_ws/src/DH116_R_URDF/DH116-R000-A1/urdf/DH116-R000-A1.urdf (robot description, URDF)
Before this commit: robot DH116-R000-A1, 17 links, 16 joints
Links:
- removed link base_link
- removed link finger11_link
- removed link finger12_link
- removed link finger13_link
- removed link finger14_link
- removed link finger21_link
- removed link finger22_link
- removed link finger23_link
- removed link finger31_link
- removed link finger32_link
- removed link finger33_link
- removed link finger41_link
- removed link finger42_link
- removed link finger43_link
- removed link finger51_link
- removed link finger52_link
- removed link finger53_link
- added link R_base_link, mass 0.10866; collision mesh filename=R_package://DH116-R000-A1/meshes/base_link.STL; visual mesh filename=R_package://DH116-R000-A1/meshes/base_link.STL
- added link R_finger11_link, mass 0.010254; collision mesh filename=R_package://DH116-R000-A1/meshes/finger11_link.STL; visual mesh filename=R_package://DH116-R000-A1/meshes/finger11_link.STL
- added link R_finger12_link, mass 0.010145; collision mesh filename=R_package://DH116-R000-A1/meshes/finger12_link.STL; visual mesh filename=R_package://DH116-R000-A1/meshes/finger12_link.STL
- added link R_finger13_link, mass 0.020548; collision mesh filename=R_package://DH116-R000-A1/meshes/finger13_link.STL; visual mesh filename=R_package://DH116-R000-A1/meshes/finger13_link.STL
- added link R_finger14_link, mass 0.00064654; collision mesh filename=R_package://DH116-R000-A1/meshes/finger14_link.STL; visual mesh filename=R_package://DH116-R000-A1/meshes/finger14_link.STL
- added link R_finger21_link, mass 0.0067143; collision mesh filename=R_package://DH116-R000-A1/meshes/finger21_link.STL; visual mesh filename=R_package://DH116-R000-A1/meshes/finger21_link.STL
- added link R_finger22_link, mass 0.014789; collision mesh filename=R_package://DH116-R000-A1/meshes/finger22_link.STL; visual mesh filename=R_package://DH116-R000-A1/meshes/finger22_link.STL
- added link R_finger23_link, mass 0.00083419; collision mesh filename=R_package://DH116-R000-A1/meshes/finger23_link.STL; visual mesh filename=R_package://DH116-R000-A1/meshes/finger23_link.STL
- added link R_finger31_link, mass 0.0067141; collision mesh filename=R_package://DH116-R000-A1/meshes/finger31_link.STL; visual mesh filename=R_package://DH116-R000-A1/meshes/finger31_link.STL
- added link R_finger32_link, mass 0.017444; collision mesh filename=R_package://DH116-R000-A1/meshes/finger32_link.STL; visual mesh filename=R_package://DH116-R000-A1/meshes/finger32_link.STL
- added link R_finger33_link, mass 0.00083416; collision mesh filename=R_package://DH116-R000-A1/meshes/finger33_link.STL; visual mesh filename=R_package://DH116-R000-A1/meshes/finger33_link.STL
- added link R_finger41_link, mass 0.006714; collision mesh filename=R_package://DH116-R000-A1/meshes/finger41_link.STL; visual mesh filename=R_package://DH116-R000-A1/meshes/finger41_link.STL
- added link R_finger42_link, mass 0.014788; collision mesh filename=R_package://DH116-R000-A1/meshes/finger42_link.STL; visual mesh filename=R_package://DH116-R000-A1/meshes/finger42_link.STL
- added link R_finger43_link, mass 0.0008342; collision mesh filename=R_package://DH116-R000-A1/meshes/finger43_link.STL; visual mesh filename=R_package://DH116-R000-A1/meshes/finger43_link.STL
- added link R_finger51_link, mass 0.0067142; collision mesh filename=R_package://DH116-R000-A1/meshes/finger51_link.STL; visual mesh filename=R_package://DH116-R000-A1/meshes/finger51_link.STL
- added link R_finger52_link, mass 0.010445; collision mesh filename=R_package://DH116-R000-A1/meshes/finger52_link.STL; visual mesh filename=R_package://DH116-R000-A1/meshes/finger52_link.STL
- added link R_finger53_link, mass 0.00059177; collision mesh filename=R_package://DH116-R000-A1/meshes/finger53_link.STL; visual mesh filename=R_package://DH116-R000-A1/meshes/finger53_link.STL
Joints:
- removed joint finger11
- removed joint finger12
- removed joint finger13
- removed joint finger14
- removed joint finger21
- removed joint finger22
- removed joint finger23
- removed joint finger31
- removed joint finger32
- removed joint finger33
- removed joint finger41
- removed joint finger42
- removed joint finger43
- removed joint finger51
- removed joint finger52
- removed joint finger53
- added joint R_finger11: type revolute, parent R_base_link, child R_finger11_link, origin xyz=0.018 0.021747 0.043279 rpy=-0.087266 0 0, axis 0 0 -1, limit lower=-1.57 upper=1.57 effort=0 velocity=0
- added joint R_finger12: type revolute, parent R_finger11_link, child R_finger12_link, origin xyz=0.018876 0.0049375 -0.0056093 rpy=0 0.95149 0.25585, axis 0 -1 0, limit lower=0 upper=1.57 effort=0 velocity=0
- added joint R_finger13: type revolute, parent R_finger12_link, child R_finger13_link, origin xyz=0 0 0.045 rpy=0 0 0, axis 0 -1 0, limit lower=0 upper=1.57 effort=0 velocity=0
- added joint R_finger14: type fixed, parent R_finger13_link, child R_finger14_link, origin xyz=0 0 0 rpy=0 0 0, axis 0 0 0, limit lower=0 upper=1.57 effort=0 velocity=0
- added joint R_finger21: type revolute, parent R_base_link, child R_finger21_link, origin xyz=-0.011581 0.031971 0.10003 rpy=-0.052657 0.10625 -0.0055894, axis 0 1 0, limit lower=0 upper=1.57 effort=0 velocity=0
- added joint R_finger22: type revolute, parent R_finger21_link, child R_finger22_link, origin xyz=0 0 0.035 rpy=0 0 0, axis 0 1 0, limit lower=0 upper=1.57 effort=0 velocity=0
- added joint R_finger23: type fixed, parent R_finger22_link, child R_finger23_link, origin xyz=0 0 0 rpy=0 0 0, axis 0 0 0, limit lower=0 upper=1.57 effort=0 velocity=0
- added joint R_finger31: type revolute, parent R_base_link, child R_finger31_link, origin xyz=-0.013501 0.0105 0.10286 rpy=0 0.10214 0, axis 0 1 0, limit lower=0 upper=1.57 effort=0 velocity=0
- added joint R_finger32: type revolute, parent R_finger31_link, child R_finger32_link, origin xyz=0 0 0.035 rpy=0 0 0, axis 0 1 0, limit lower=0 upper=1.57 effort=0 velocity=0
- added joint R_finger33: type fixed, parent R_finger32_link, child R_finger33_link, origin xyz=0 0 0 rpy=0 0 0, axis 0 0 0, limit lower=0 upper=1.57 effort=0 velocity=0
- added joint R_finger41: type revolute, parent R_base_link, child R_finger41_link, origin xyz=-0.015081 -0.010971 0.10183 rpy=0.052889 0.14148 0.0074648, axis 0 1 0, limit lower=0 upper=1.57 effort=0 velocity=0
- added joint R_finger42: type revolute, parent R_finger41_link, child R_finger42_link, origin xyz=0 0 0.035 rpy=0 0 0, axis 0 1 0, limit lower=0 upper=1.57 effort=0 velocity=0
- added joint R_finger43: type fixed, parent R_finger42_link, child R_finger43_link, origin xyz=0 0 0 rpy=0 0 0, axis 0 0 0, limit lower=0 upper=1.57 effort=0 velocity=0
- added joint R_finger51: type revolute, parent R_base_link, child R_finger51_link, origin xyz=-0.013081 -0.032156 0.097798 rpy=0.078754 0.073706 0.0058113, axis 0 1 0, limit lower=0 upper=1.57 effort=0 velocity=0
- added joint R_finger52: type revolute, parent R_finger51_link, child R_finger52_link, origin xyz=0 0 0.035 rpy=0 0 0, axis 0 1 0, limit lower=0 upper=1.57 effort=0 velocity=0
- added joint R_finger53: type fixed, parent R_finger52_link, child R_finger53_link, origin xyz=0 0 0 rpy=0 0 0, axis 0 0 0, limit lower=0 upper=1.57 effort=0 velocity=0
