Commit message: Fix package naming, resolve build warnings, and save current progress

File: ros2_ws/src/DH116_L_URDF/dh116_l000_a1/urdf/DH116-L000-A1.urdf (robot description, URDF)
Before this commit: robot L_DH116-L000-A1, 17 links, 16 joints
Links:
- link L_base_link: geometry collision mesh filename=package://dh116_l000_a1/meshes/base_link.STL; visual mesh filename=package://dh116_l000_a1/meshes/base_link.STL
- link L_finger11_Link: geometry collision mesh filename=package://dh116_l000_a1/meshes/finger11_Link.STL; visual mesh filename=package://dh116_l000_a1/meshes/finger11_Link.STL
- link L_finger12_Link: geometry collision mesh filename=package://dh116_l000_a1/meshes/finger12_Link.STL; visual mesh filename=package://dh116_l000_a1/meshes/finger12_Link.STL
- link L_finger13_Link: geometry collision mesh filename=package://dh116_l000_a1/meshes/finger13_Link.STL; visual mesh filename=package://dh116_l000_a1/meshes/finger13_Link.STL
- link L_finger14_Link: geometry collision mesh filename=package://dh116_l000_a1/meshes/finger14_Link.STL; visual mesh filename=package://dh116_l000_a1/meshes/finger14_Link.STL
- link L_finger21_Link: geometry collision mesh filename=package://dh116_l000_a1/meshes/finger21_Link.STL; visual mesh filename=package://dh116_l000_a1/meshes/finger21_Link.STL
- link L_finger22_Link: geometry collision mesh filename=package://dh116_l000_a1/meshes/finger22_Link.STL; visual mesh filename=package://dh116_l000_a1/meshes/finger22_Link.STL
- link L_finger23_Link: geometry collision mesh filename=package://dh116_l000_a1/meshes/finger23_Link.STL; visual mesh filename=package://dh116_l000_a1/meshes/finger23_Link.STL
- link L_finger31_Link: geometry collision mesh filename=package://dh116_l000_a1/meshes/finger31_Link.STL; visual mesh filename=package://dh116_l000_a1/meshes/finger31_Link.STL
- link L_finger32_Link: geometry collision mesh filename=package://dh116_l000_a1/meshes/finger32_Link.STL; visual mesh filename=package://dh116_l000_a1/meshes/finger32_Link.STL
- link L_finger33_Link: geometry collision mesh filename=package://dh116_l000_a1/meshes/finger33_Link.STL; visual mesh filename=package://dh116_l000_a1/meshes/finger33_Link.STL
- link L_finger41_Link: geometry collision mesh filename=package://dh116_l000_a1/meshes/finger41_Link.STL; visual mesh filename=package://dh116_l000_a1/meshes/finger41_Link.STL
- link L_finger42_Link: geometry collision mesh filename=package://dh116_l000_a1/meshes/finger42_Link.STL; visual mesh filename=package://dh116_l000_a1/meshes/finger42_Link.STL
- link L_finger43_Link: geometry collision mesh filename=package://dh116_l000_a1/meshes/finger43_Link.STL; visual mesh filename=package://dh116_l000_a1/meshes/finger43_Link.STL
- link L_finger51_Link: geometry collision mesh filename=package://dh116_l000_a1/meshes/finger51_Link.STL; visual mesh filename=package://dh116_l000_a1/meshes/finger51_Link.STL
- link L_finger52_Link: geometry collision mesh filename=package://dh116_l000_a1/meshes/finger52_Link.STL; visual mesh filename=package://dh116_l000_a1/meshes/finger52_Link.STL
- link L_finger53_Link: geometry collision mesh filename=package://dh116_l000_a1/meshes/finger53_Link.STL; visual mesh filename=package://dh116_l000_a1/meshes/finger53_Link.STL

File: ros2_ws/src/DH116_R_URDF/dh116_r000_a1/urdf/DH116-R000-A1.urdf (robot description, URDF)
Before this commit: robot R_DH116-R000-A1, 17 links, 16 joints
Links:
- link R_base_link: geometry collision mesh filename=package://dh116_r000_a1/meshes/base_link.STL; visual mesh filename=package://dh116_r000_a1/meshes/base_link.STL
- link R_finger11_link: geometry collision mesh filename=package://dh116_r000_a1/meshes/finger11_link.STL; visual mesh filename=package://dh116_r000_a1/meshes/finger11_link.STL
- link R_finger12_link: geometry collision mesh filename=package://dh116_r000_a1/meshes/finger12_link.STL; visual mesh filename=package://dh116_r000_a1/meshes/finger12_link.STL
- link R_finger13_link: geometry collision mesh filename=package://dh116_r000_a1/meshes/finger13_link.STL; visual mesh filename=package://dh116_r000_a1/meshes/finger13_link.STL
- link R_finger14_link: geometry collision mesh filename=package://dh116_r000_a1/meshes/finger14_link.STL; visual mesh filename=package://dh116_r000_a1/meshes/finger14_link.STL
- link R_finger21_link: geometry collision mesh filename=package://dh116_r000_a1/meshes/finger21_link.STL; visual mesh filename=package://dh116_r000_a1/meshes/finger21_link.STL
- link R_finger22_link: geometry collision mesh filename=package://dh116_r000_a1/meshes/finger22_link.STL; visual mesh filename=package://dh116_r000_a1/meshes/finger22_link.STL
- link R_finger23_link: geometry collision mesh filename=package://dh116_r000_a1/meshes/finger23_link.STL; visual mesh filename=package://dh116_r000_a1/meshes/finger23_link.STL
- link R_finger31_link: geometry collision mesh filename=package://dh116_r000_a1/meshes/finger31_link.STL; visual mesh filename=package://dh116_r000_a1/meshes/finger31_link.STL
- link R_finger32_link: geometry collision mesh filename=package://dh116_r000_a1/meshes/finger32_link.STL; visual mesh filename=package://dh116_r000_a1/meshes/finger32_link.STL
- link R_finger33_link: geometry collision mesh filename=package://dh116_r000_a1/meshes/finger33_link.STL; visual mesh filename=package://dh116_r000_a1/meshes/finger33_link.STL
- link R_finger41_link: geometry collision mesh filename=package://dh116_r000_a1/meshes/finger41_link.STL; visual mesh filename=package://dh116_r000_a1/meshes/finger41_link.STL
- link R_finger42_link: geometry collision mesh filename=package://dh116_r000_a1/meshes/finger42_link.STL; visual mesh filename=package://dh116_r000_a1/meshes/finger42_link.STL
- link R_finger43_link: geometry collision mesh filename=package://dh116_r000_a1/meshes/finger43_link.STL; visual mesh filename=package://dh116_r000_a1/meshes/finger43_link.STL
- link R_finger51_link: geometry collision mesh filename=package://dh116_r000_a1/meshes/finger51_link.STL; visual mesh filename=package://dh116_r000_a1/meshes/finger51_link.STL
- link R_finger52_link: geometry collision mesh filename=package://dh116_r000_a1/meshes/finger52_link.STL; visual mesh filename=package://dh116_r000_a1/meshes/finger52_link.STL
- link R_finger53_link: geometry collision mesh filename=package://dh116_r000_a1/meshes/finger53_link.STL; visual mesh filename=package://dh116_r000_a1/meshes/finger53_link.STL
